File: Models and Schematics/Montessori_Schematic.kicad_sch (KiCad schematic)
At the start: 5 parts, among them U1 DFR0478

Commit message: Updated Models and Schematics
Connections:
- net A0: now reaches U1.19 (A0/IO36)
- net A0: now also R1.2, R2.2, R3.1, R4.1
- removed net A3: R1.2, R4.1, U1.22 (A3/IO35)
- removed net A4: R2.2, R3.1, U1.23 (A4/IO15)
Changed lines of the file:
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@@
+	(wire
+		(pts
+			(xy 78.74 30.48) (xy 86.36 30.48)
+		)
+		(stroke
+			(width 0)
+			(type default)
+		)
+	)
 	(wire
 		(pts
@@
 	(wire
 		(pts
-			(xy 78.74 38.1) (xy 86.36 38.1)
-		)
-		(stroke
-			(width 0)
-			(type default)
-		)
-	)
-	(wire
-		(pts
 			(xy 110.49 26.67) (xy 127 26.67)
 		)
@@
 		(pts
 			(xy 110.49 34.29) (xy 110.49 38.1)
-		)
-		(stroke
-			(width 0)
-			(type default)
-		)
-	)
-	(wire
-		(pts
-			(xy 78.74 40.64) (xy 86.36 40.64)
 		)
 		(stroke
@@
 		)
 	)
-	(label "A3"
+	(label "A0"
 		(at 114.3 38.1 0)
 		(fields_autoplaced yes)
@@
 		)
 	)
-	(label "A4"
+	(label "A0"
 		(at 130.81 38.1 0)
 		(fields_autoplaced yes)
@@
 		)
 	)
+	(label "A0"
+		(at 86.36 30.48 0)
+		(fields_autoplaced yes)
+		(effects
+			(font
+				(size 1.27 1.27)
+			)
+			(justify left bottom)
+		)
+	)
 	(label "GND"
 		(at 21.59 66.04 0)
 		(fields_autoplaced yes)
 		(effects
-			(font
-				(size 1.27 1.27)
-			)
-			(justify left bottom)
-		)
-	)
-	(label "A3"
-		(at 86.36 38.1 0)
-		(fields_autoplaced yes)
-		(effects
-			(font
-				(size 1.27 1.27)
-			)
-			(justify left bottom)
-		)
-	)
-	(label "A4"
-		(at 86.36 40.64 0)
-		(fields_autoplaced yes)
-		(effects
